File: hardware/GH-4DEV/greenhouse.kicad_sch (KiCad schematic)
At the start: 164 parts, among them K1 OMRON G5LE, K2 OMRON G5LE, K3 OMRON G5LE, K4 OMRON G5LE, K5 OMRON G5LE, K6 OMRON G5LE, K7 OMRON G5LE, U1 PC847, U2 PC817, U3 MOC3052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

Commit message: fix: update hw to kicad 7, fix capacitor placement in 4.0dev
Other:
- moved on the sheet: C35, R13, R19, R23, R55, R56, R57, R58, R59, R63, SA1A, SA1B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

Commit message: Мелкие правки в железе и диммере
Parts:
- removed HL8: RL6, LED_SMD:LED_0805_2012Metric_Pad1.15x1.40mm_HandSolder, symbol GOST_Opto:LED1
- removed K7: OMRON G5LE, Relay_THT:Relay_SPDT_Omron-G5LE-1, symbol GOST_Relays:OMRON_G5LE
- removed X14: RELAY6, TerminalBlock:TerminalBlock_bornier-3_P5.08mm, symbol GOST_Connectors_List:CONN_LIST_03_L
- added C38: 0,01/400V, Capacitor_THT:C_Rect_L13.0mm_W5.0mm_P10.00mm_FKS3_FKP3_MKS4, symbol GOST_Capacitors:CAPACITOR
- added HL8: STATUS0, LED_SMD:LED_0805_2012Metric_Pad1.15x1.40mm_HandSolder, symbol GOST_Opto:LED2
- added HL9: STATUS1, LED_SMD:LED_0805_2012Metric_Pad1.15x1.40mm_HandSolder, symbol GOST_Opto:LED2
- added R60: 33, Resistor_THT:R_Axial_DIN0614_L14.3mm_D5.7mm_P20.32mm_Horizontal, symbol GOST_Resistors:RESISTOR_1000
- added R61, R62: 820, Resistor_SMD:R_0805_2012Metric_Pad1.20x1.40mm_HandSolder, symbol GOST_Resistors:RESISTOR
- added R64, R65: 1,0, Resistor_THT:R_Axial_DIN0309_L9.0mm_D3.2mm_P2.54mm_Vertical, symbol GOST_Resistors:RESISTOR_0500
- added U4: MOC3052, Package_DIP:DIP-6_W7.62mm_LongPads, symbol GOST_Opto:OPTOTRIAC
- added VS2: BT139-600D, Package_TO_SOT_THT:TO-220-3_Vertical, symbol GOST_Thyristors:TRIAC
- added X19: DIMMER 1, TerminalBlock:TerminalBlock_bornier-2_P5.08mm, symbol GOST_Connectors_List:CONN_LIST_02_L
- R50: value 10k -> 330
- R54: value 820 -> 330
Connections:
- net +5V: no longer R54.1 (L)
- net ACL: now also R64.1 (L), R65.1 (L); no longer C35.1, VS1.1 (K)
- net ACN: now also X19.1
- net GND: now also DA6.7 (7B), HL8.1 (K), HL9.1 (K), U4.2; no longer R50.2 (R)
- net DIM1_CTRL: now reaches DD1.37 (IO23)
- net DIM1_CTRL: now also R50.1 (L)
- net STATUS_LED1: now reaches DD2.11 (P07)
- net STATUS_LED1: now also R62.1 (L)
- net at R54.2 (R): now also U4.6
- removed net RL6: DA6.7 (7B), DD2.10 (P06), R50.1 (L)
- net RLD6: no longer names the net of DA6.10 (7C)
- new net: R50.2 (R), U4.1
- new net: C38.1, R65.2 (R), VS2.1 (K)
- new net: C38.2, R60.1 (L)
- new net: HL8.2 (A), R61.2 (R)
- new net: HL9.2 (A), R62.2 (R)
- new net: C35.1, R64.2 (R), VS1.1 (K)
- new net: U4.4, VS2.3 (G)
- new net DIM1_OUT: R54.1 (L), R60.2 (R), VS2.2 (A), X19.2
- new net STATUS_LED0: DD2.10 (P06), R61.1 (L)
- no-connect marks 17 -> 16
Other:
- moved on the sheet: C1, C10, C11, C12, C13, C14, C15, C16, C17, C18, C19, C2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
