File: hardware/pH-meter/ph_meter.kicad_pcb (KiCad board)
At the start: 2 copper layers, 38 x 17 mm, 19 parts, among them X1 GLASS pH PROBE, X2 MCU

Commit message: Мелкие правки в железе и диммере
Parts:
- moved C2 1.00 mm to (103.5, 87.2)
- moved DA2 0.46 mm to (98.1, 86.7)
- moved C3 0.29 mm to (98.7, 79.2)
- moved DA1 0.15 mm to (98.1, 82.5)
Routing:
- net GND: track 1.47 -> 11.0 mm, vias 15 -> 11
- net +3V3: track 50.3 -> 55.4 mm
- net SCL: track 9.79 -> 9.24 mm
- net Net-(DA2.1--): track 37.6 -> 38.1 mm
- removed copper zone on F.Cu, net GND
